File: Hardware/drone/drone.kicad_pcb (KiCad board)
At the start: 2 copper layers, 11 parts, among them M1 Motor_DC, M2 Motor_DC, M3 Motor_DC, M4 Motor_DC, U1 ESP32-DEVKITC, U2 MPU6050 DevKit, U3 HW_611, U4 DRV8833, U5 DRV8833, U6 MT3608

Commit message: PCB design v1.0
Parts:
- moved M3 90.4 mm to (144.7, 154.7)
- moved M4 81.0 mm to (69.9, 151.7)
- moved U3 66.0 mm to (122.9, 113.7)
- moved U1 62.9 mm to (87.0, 101.2)
- moved U4 53.0 mm to (79.4, 116.9), turned to 180 degrees
- moved U5 51.6 mm to (79.4, 139.9), turned to 180 degrees
- moved U2 50.6 mm to (132.8, 119.3)
- moved M1 48.6 mm to (69.9, 91.7)
- moved M2 47.0 mm to (145.9, 91.7)
- moved BT1 32.8 mm to (151.8, 126.7), turned to -90 degrees
- moved U6 25.6 mm to (136.8, 139.7), turned to 0 degrees
Connections:
- U1 pad 10: unconnected-(U1-IO26-Pad10) -> PWM_3
- U1 pad 11: unconnected-(U1-IO27-Pad11) -> PWM_4
- U1 pad 24: PWM_3 -> unconnected-(U1-IO2-Pad24)
- U1 pad 25: PWM_4 -> unconnected-(U1-IO0-Pad25)
- U1 pad 27: PWM_1 -> unconnected-(U1-IO16-Pad27)
- U1 pad 28: PWM_2 -> unconnected-(U1-IO17-Pad28)
- U1 pad 5: unconnected-(U1-IO34-Pad5) -> PWM_1
- U1 pad 6: unconnected-(U1-IO35-Pad6) -> PWM_2
Routing:
- net GND: track 0.00 -> 155.2 mm
- net VBAT: track 0.00 -> 139.9 mm, vias 0 -> 3
- net MOTOR_2+: track 0.00 -> 94.1 mm
- net MOTOR_3-: track 0.00 -> 93.9 mm
- net MOTOR_2-: track 0.00 -> 88.0 mm
- net MOTOR_3+: track 0.00 -> 87.7 mm
- net +3.3V: track 0.00 -> 47.2 mm
- net +5V: track 0.00 -> 46.6 mm
- net SENSOR_INT: track 0.00 -> 29.9 mm
- net MOTOR_1+: track 0.00 -> 28.6 mm
- net MOTOR_4-: track 0.00 -> 27.8 mm
- net MOTOR_4+: track 0.00 -> 27.4 mm
- net MOTOR_1-: track 0.00 -> 27.3 mm
- net SENSOR_DATA: track 0.00 -> 22.6 mm
- net SENSOR_CLK: track 0.00 -> 20.5 mm
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