File: Hardware/drone/drone.kicad_sch (KiCad schematic)
At the start: 9 parts, among them M1 Motor_DC, M2 Motor_DC, M3 Motor_DC, M4 Motor_DC, U1 ESP32-DEVKITC, U2 MPU6050 DevKit, U3 HW_611, U4 DRV8833, U5 DRV8833

Commit message: Hardware schematic update.
Parts:
- added BT1: 3.7V, symbol Device:Battery_Cell
- added U6: MT3608, symbol Custom_drone:MT3608
Connections:
- net +5V: now also U6. (VIN-)
- net GND: now also U2. (INT), U3. (SDD), U4. (ULT), U5. (ULT), U6. (VIN-)
- net MOTOR_3+: now reaches M3.1 (+)
- net MOTOR_3+: now also U5. (ULT)
- net MOTOR_3-: now reaches M3.2 (-)
- net MOTOR_3-: now also U5. (ULT)
- net SENSOR_DATA: now reaches U3. (SDD)
- net SENSOR_DATA: now also U1.33 (IO21), U2. (INT)
- net MOTOR_4-: now reaches M4.1 (+)
- net MOTOR_4-: now also U5. (ULT)
- net MOTOR_4+: now reaches M4.2 (-)
- net MOTOR_4+: now also U5. (ULT)
- net MOTOR_1+: now reaches M1.1 (+)
- net MOTOR_1+: now also U4. (ULT)
- net MOTOR_1-: now reaches M1.2 (-)
- net MOTOR_1-: now also U4. (ULT)
- net VBAT: now reaches U4. (ULT)
- net VBAT: now also U5. (ULT), BT1.1 (+), U6. (VIN-)
- net SENSOR_INT: now reaches U2. (INT)
- net SENSOR_INT: now also U1.26 (IO4)
- net MOTOR_2-: now reaches M2.1 (+)
- net MOTOR_2-: now also U4. (ULT)
- net MOTOR_2+: now reaches M2.2 (-)
- net MOTOR_2+: now also U4. (ULT)
- net +3.3V: now reaches U1.1 (3V3)
- net +3.3V: now also U2. (INT), U3. (SDD)
- net PWM_3: now reaches U1.24 (IO2)
- net PWM_3: now also U5. (ULT)
- net PWM_4: now reaches U1.25 (IO0)
- net PWM_4: now also U5. (ULT)
- net PWM_1: now reaches U1.27 (IO16)
- net PWM_1: now also U4. (ULT)
- net PWM_2: now reaches U1.28 (IO17)
- net PWM_2: now also U4. (ULT)
- net SENSOR_CLK: now reaches U1.36 (IO22)
- net SENSOR_CLK: now also U2. (INT), U3. (SDD)
- new net: BT1.2 (-), U6. (VIN-)
- no-connect marks 0 -> 9
Other:
- moved on the sheet: M1, M2, M3, M4, U1, U2, U3, U4, U5

Commit message: Footprints updated.
Parts:
- BT1: footprint (none) -> Connector_PinHeader_2.54mm:PinHeader_1x02_P2.54mm_Vertical
- M1, M2, M3, M4: footprint (none) -> Resistor_THT:R_Axial_DIN0516_L15.5mm_D5.0mm_P5.08mm_Vertical
- U1: footprint ESP32-DEVKITC:MODULE_ESP32-DEVKITC -> esp32:ESP32-DevKitC
- U2: footprint (none) -> usini:module_mpu6050
- U3: footprint (none) -> usini:module_bme280
- U4, U5: footprint (none) -> usini:DIP-12_W15.24mm_LongPads
- U6: footprint (none) -> mt3608:hw-045
Connections:
- net +3.3V: now also U2.1 (VCC), U3.1 (VCC); no longer U2. (INT), U3. (SDD)
- net +5V: now also U6.2 (VOUT+); no longer U6. (VIN-)
- net GND: now also U2.2 (GND), U3.2 (GND), U4.1 (IN4), U4.3 (GND), U4.5 (IN2), U5.1 (IN4), U5.3 (GND), U5.5 (IN2), U6.1 (VOUT-); no longer U2. (INT), U3. (SDD), U4. (ULT), U5. (ULT), U6. (VIN-)
- net MOTOR_1+: now also U4.8 (OUT1); no longer U4. (ULT)
- net MOTOR_1-: now also U4.9 (OUT2); no longer U4. (ULT)
- net MOTOR_2+: now also U4.10 (OUT3); no longer U4. (ULT)
- net MOTOR_2-: now also U4.11 (OUT4); no longer U4. (ULT)
- net MOTOR_3+: now also U5.8 (OUT1); no longer U5. (ULT)
- net MOTOR_3-: now also U5.9 (OUT2); no longer U5. (ULT)
- net MOTOR_4+: now also U5.10 (OUT3); no longer U5. (ULT)
- net MOTOR_4-: now also U5.11 (OUT4); no longer U5. (ULT)
- net PWM_1: now also U4.6 (IN1); no longer U4. (ULT)
- net PWM_2: now also U4.2 (IN3); no longer U4. (ULT)
- net PWM_3: now also U5.6 (IN1); no longer U5. (ULT)
- net PWM_4: now also U5.2 (IN3); no longer U5. (ULT)
- net SENSOR_CLK: now also U2.3 (SCL), U3.3 (SCL); no longer U2. (INT), U3. (SDD)
- net SENSOR_DATA: now also U2.4 (SDA), U3.4 (SDA); no longer U2. (INT), U3. (SDD)
- net SENSOR_INT: now also U2.8 (INT); no longer U2. (INT)
- net VBAT: now also U4.4 (VCC), U5.4 (VCC), U6.3 (VIN+); no longer U4. (ULT), U5. (ULT), U6. (VIN-)
- net at BT1.2 (-): now also U6.4 (VIN-); no longer U6. (VIN-)
- no-connect marks 9 -> 35
Other:
- moved on the sheet: BT1
Changed lines of the file:
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@@
 	)
 	(no_connect
+		(at 215.9 129.54)
+	)
+	(no_connect
+		(at 175.26 124.46)
+	)
+	(no_connect
 		(at 63.5 123.19)
 	)
 	(no_connect
+		(at 175.26 88.9)
+	)
+	(no_connect
+		(at 175.26 116.84)
+	)
+	(no_connect
+		(at 175.26 101.6)
+	)
+	(no_connect
+		(at 215.9 93.98)
+	)
+	(no_connect
+		(at 215.9 109.22)
+	)
+	(no_connect
+		(at 175.26 106.68)
+	)
+	(no_connect
 		(at 128.27 48.26)
 	)
 	(no_connect
+		(at 215.9 106.68)
+	)
+	(no_connect
+		(at 215.9 132.08)
+	)
+	(no_connect
+		(at 175.26 129.54)
+	)
+	(no_connect
 		(at 63.5 78.74)
 	)
 	(no_connect
+		(at 215.9 127)
+	)
+	(no_connect
+		(at 175.26 127)
+	)
+	(no_connect
+		(at 215.9 124.46)
+	)
+	(no_connect
+		(at 175.26 114.3)
+	)
+	(no_connect
+		(at 175.26 99.06)
+	)
+	(no_connect
+		(at 175.26 104.14)
+	)
+	(no_connect
+		(at 175.26 111.76)
+	)
+	(no_connect
 		(at 67.31 44.45)
 	)
 	(no_connect
+		(at 215.9 88.9)
+	)
+	(no_connect
 		(at 128.27 45.72)
 	)
 	(no_connect
+		(at 215.9 104.14)
+	)
+	(no_connect
+		(at 175.26 109.22)
+	)
+	(no_connect
+		(at 175.26 93.98)
+	)
+	(no_connect
 		(at 67.31 46.99)
 	)
 	(no_connect
+		(at 175.26 91.44)
+	)
+	(no_connect
 		(at 67.31 41.91)
 	)
 	(no_connect
+		(at 215.9 96.52)
+	)
+	(no_connect
+		(at 175.26 121.92)
+	)
+	(no_connect
+		(at 175.26 96.52)
+	)
+	(no_connect
 		(at 63.5 91.44)
 	)
@@
 	(wire
 		(pts
+			(xy 215.9 34.29) (xy 215.9 35.56)
+		)
+		(stroke
+			(width 0)
+			(type default)
+		)
+	)
+	(wire
+		(pts
 			(xy 215.9 116.84) (xy 222.25 116.84)
 		)
@@
 	(wire
 		(pts
-			(xy 215.9 43.18) (xy 208.28 43.18)
+			(xy 219.71 43.18) (xy 208.28 43.18)
+		)
+		(stroke
+			(width 0)
+			(type default)
+		)
+	)
+	(wire
+		(pts
+			(xy 219.71 35.56) (xy 215.9 35.56)
 		)
 		(stroke
@@
 			)
 		)
-		(property "Footprint" ""
+		(property "Footprint" "Resistor_THT:R_Axial_DIN0516_L15.5mm_D5.0mm_P5.08mm_Vertical"
 			(at 87.63 163.576 0)
 			(effects
@@
 			)
 		)
-		(property "Footprint" ""
+		(property "Footprint" "usini:module_bme280"
 			(at 120.65 41.91 0)
 			(effects
@@
 			)
 		)
-		(pin ""
+		(pin "4"
 		)
-		(pin ""
+		(pin "6"
 		)
-		(pin ""
+		(pin "2"
 		)
-		(pin ""
+		(pin "1"
 		)
-		(pin ""
+		(pin "3"
 		)
-		(pin ""
+		(pin "5"
 		)
 		(instances
@@
 			)
 		)
-		(property "Footprint" ""
+		(property "Footprint" "mt3608:hw-045"
 			(at 196.85 39.37 0)
 			(effects
@@
 			)
 		)
-		(pin ""
+		(pin "1"
 		)
-		(pin ""
+		(pin "2"
 		)
-		(pin ""
+		(pin "4"
 		)
-		(pin ""
+		(pin "3"
 		)
 		(instances
@@
 			)
 		)
-		(property "Footprint" ""
+		(property "Footprint" "Resistor_THT:R_Axial_DIN0516_L15.5mm_D5.0mm_P5.08mm_Vertical"
 			(at 107.95 163.576 0)
 			(effects
@@
 	(symbol
 		(lib_id "power:VCC")
-		(at 215.9 35.56 0)
+		(at 215.9 34.29 0)
 		(unit 1)
 		(exclude_from_sim no)
@@
 		(fields_autoplaced yes)
 		(property "Reference" "#PWR013"
-			(at 215.9 39.37 0)
+			(at 215.9 38.1 0)
 			(effects
 				(font
@@
 		)
 		(property "Value" "VBAT"
-			(at 215.9 30.48 0)
+			(at 215.9 29.21 0)
 			(effects
 				(font
@@
 		)
 		(property "Footprint" ""
-			(at 215.9 35.56 0)
+			(at 215.9 34.29 0)
 			(effects
 				(font
@@
 		)
 		(property "Datasheet" ""
-			(at 215.9 35.56 0)
+			(at 215.9 34.29 0)
 			(effects
 				(font
@@
 		)
 		(property "Description" "Power symbol creates a global label with name \"VCC\""
-			(at 215.9 35.56 0)
+			(at 215.9 34.29 0)
 			(effects
 				(font
@@
 			)
 		)
-		(property "Footprint" ""
+		(property "Footprint" "Resistor_THT:R_Axial_DIN0516_L15.5mm_D5.0mm_P5.08mm_Vertical"
 			(at 48.26 163.576 0)
 			(effects
@@
 			)
 		)
-		(property "Footprint" ""
+		(property "Footprint" "usini:DIP-12_W15.24mm_LongPads"
 			(at 54.61 85.09 0)
 			(effects
@@
 			)
 		)
-		(pin ""
+		(pin "5"
 		)
-		(pin ""
+		(pin "1"
 		)
-		(pin ""
+		(pin "8"
 		)
-		(pin ""
+		(pin "12"
 		)
-		(pin ""
+		(pin "3"
 		)
-		(pin ""
+		(pin "11"
 		)
-		(pin ""
+		(pin "10"
 		)
-		(pin ""
+		(pin "6"
 		)
-		(pin ""
+		(pin "7"
 		)
-		(pin ""
+		(pin "9"
 		)
-		(pin ""
+		(pin "4"
 		)
-		(pin ""
+		(pin "2"
 		)
 		(instances
@@
 			)
 		)
-		(property "Footprint" ""
+		(property "Footprint" "usini:module_mpu6050"
 			(at 54.61 40.64 0)
 			(effects
@@
 			)
 		)
-		(pin ""
+		(pin "2"
 		)
-		(pin ""
+		(pin "7"
 		)
-		(pin ""
+		(pin "3"
 		)
-		(pin ""
+		(pin "6"
 		)
-		(pin ""
+		(pin "1"
 		)
-		(pin ""
+		(pin "5"
 		)
-		(pin ""
+		(pin "4"
 		)
-		(pin ""
+		(pin "8"
 		)
 		(instances
@@
 	(symbol
 		(lib_id "Device:Battery_Cell")
-		(at 215.9 40.64 0)
+		(at 219.71 40.64 0)
 		(unit 1)
 		(exclude_from_sim no)
@@
 		(fields_autoplaced yes)
 		(property "Reference" "BT1"
-			(at 219.71 37.5284 0)
+			(at 223.52 37.5284 0)
 			(effects
 				(font
@@
 		)
 		(property "Value" "3.7V"
-			(at 219.71 40.0684 0)
+			(at 223.52 40.0684 0)
 			(effects
 				(font
@@
 			)
 		)
-		(property "Footprint" ""
-			(at 215.9 39.116 90)
+		(property "Footprint" "Connector_PinHeader_2.54mm:PinHeader_1x02_P2.54mm_Vertical"
+			(at 219.71 39.116 90)
 			(effects
 				(font
@@
 		)
 		(property "Datasheet" "~"
-			(at 215.9 39.116 90)
+			(at 219.71 39.116 90)
 			(effects
 				(font
@@
 		)
 		(property "Description" "Single-cell battery"
-			(at 215.9 40.64 0)
+			(at 219.71 40.64 0)
 			(effects
 				(font
@@
 		)
 		(property "Sim.Device" "V"
-			(at 215.9 40.64 0)
+			(at 219.71 40.64 0)
 			(effects
 				(font
@@
 		)
 		(property "Sim.Type" "DC"
-			(at 215.9 40.64 0)
+			(at 219.71 40.64 0)
 			(effects
 				(font
@@
 		)
 		(property "Sim.Pins" "1=+ 2=-"
-			(at 215.9 40.64 0)
+			(at 219.71 40.64 0)
 			(effects
 				(font
@@
 			)
 		)
-		(property "Footprint" ""
+		(property "Footprint" "Resistor_THT:R_Axial_DIN0516_L15.5mm_D5.0mm_P5.08mm_Vertical"
 			(at 67.31 163.576 0)
 			(effects
@@
 			)
 		)
-		(property "Footprint" ""
+		(property "Footprint" "usini:DIP-12_W15.24mm_LongPads"
 			(at 54.61 116.84 0)
 			(effects
@@
 			)
 		)
-		(pin ""
+		(pin "7"
 		)
-		(pin ""
+		(pin "12"
 		)
-		(pin ""
+		(pin "8"
 		)
-		(pin ""
+		(pin "4"
 		)
-		(pin ""
+		(pin "6"
 		)
-		(pin ""
+		(pin "2"
 		)
-		(pin ""
+		(pin "5"
 		)
-		(pin ""
+		(pin "3"
 		)
-		(pin ""
+		(pin "1"
 		)
-		(pin ""
+		(pin "11"
 		)
-		(pin ""
+		(pin "9"
 		)
-		(pin ""
+		(pin "10"
 		)
 		(instances
@@
 			)
 		)
-		(property "Footprint" "ESP32-DEVKITC:MODULE_ESP32-DEVKITC"
+		(property "Footprint" "esp32:ESP32-DevKitC"
 			(at 195.58 109.22 0)
 			(effects

Commit message: PCB design v1.0
Connections:
- net PWM_1: now also U1.5 (IO34); no longer U1.27 (IO16)
- net PWM_2: now also U1.6 (IO35); no longer U1.28 (IO17)
- net PWM_3: now also U1.10 (IO26); no longer U1.24 (IO2)
- net PWM_4: now also U1.11 (IO27); no longer U1.25 (IO0)
Changed lines of the file:
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@@
+	)
+	(no_connect
+		(at 215.9 121.92)
 	)
 	(no_connect
@@
 	)
 	(no_connect
+		(at 215.9 119.38)
+	)
+	(no_connect
 		(at 128.27 48.26)
 	)
@@
 	)
 	(no_connect
-		(at 175.26 99.06)
-	)
-	(no_connect
 		(at 175.26 104.14)
 	)
 	(no_connect
-		(at 175.26 111.76)
-	)
-	(no_connect
 		(at 67.31 44.45)
 	)
 	(no_connect
+		(at 215.9 111.76)
+	)
+	(no_connect
 		(at 215.9 88.9)
 	)
@@
 	)
 	(no_connect
-		(at 175.26 109.22)
-	)
-	(no_connect
 		(at 175.26 93.98)
 	)
@@
 	)
 	(no_connect
-		(at 175.26 96.52)
+		(at 215.9 114.3)
 	)
 	(no_connect
@@
 	(wire
 		(pts
-			(xy 215.9 119.38) (xy 222.25 119.38)
+			(xy 170.18 99.06) (xy 175.26 99.06)
 		)
 		(stroke
@@
 	(wire
 		(pts
-			(xy 215.9 111.76) (xy 222.25 111.76)
+			(xy 170.18 96.52) (xy 175.26 96.52)
 		)
 		(stroke
@@
 	(wire
 		(pts
+			(xy 170.18 111.76) (xy 175.26 111.76)
+		)
+		(stroke
+			(width 0)
+			(type default)
+		)
+	)
+	(wire
+		(pts
 			(xy 215.9 86.36) (xy 220.98 86.36)
 		)
@@
 	(wire
 		(pts
+			(xy 170.18 109.22) (xy 175.26 109.22)
+		)
+		(stroke
+			(width 0)
+			(type default)
+		)
+	)
+	(wire
+		(pts
 			(xy 67.31 36.83) (xy 72.39 36.83)
 		)
@@
 	(wire
 		(pts
-			(xy 215.9 121.92) (xy 222.25 121.92)
-		)
-		(stroke
-			(width 0)
-			(type default)
-		)
-	)
-	(wire
-		(pts
-			(xy 215.9 114.3) (xy 222.25 114.3)
-		)
-		(stroke
-			(width 0)
-			(type default)
-		)
-	)
-	(wire
-		(pts
 			(xy 168.91 132.08) (xy 175.26 132.08)
 		)
@@
 		)
 	)
+	(global_label "PWM_4"
+		(shape output)
+		(at 170.18 111.76 180)
+		(fields_autoplaced yes)
+		(effects
+			(font
+				(size 1.27 1.27)
+			)
+			(justify right)
+		)
+		(property "Intersheetrefs" "${INTERSHEET_REFS}"
+			(at 160.8449 111.76 0)
+			(effects
+				(font
+					(size 1.27 1.27)
+				)
+				(justify right)
+				(hide yes)
+			)
+		)
+	)
 	(global_label "PWM_3"
 		(shape output)
-		(at 222.25 121.92 0)
-		(fields_autoplaced yes)
-		(effects
-			(font
-				(size 1.27 1.27)
-			)
-			(justify left)
-		)
-		(property "Intersheetrefs" "${INTERSHEET_REFS}"
-			(at 231.5851 121.92 0)
-			(effects
-				(font
-					(size 1.27 1.27)
-				)
-				(justify left)
+		(at 170.18 109.22 180)
+		(fields_autoplaced yes)
+		(effects
+			(font
+				(size 1.27 1.27)
+			)
+			(justify right)
+		)
+		(property "Intersheetrefs" "${INTERSHEET_REFS}"
+			(at 160.8449 109.22 0)
+			(effects
+				(font
+					(size 1.27 1.27)
+				)
+				(justify right)
 				(hide yes)
 			)
@@
 				)
 				(justify left)
+				(hide yes)
+			)
+		)
+	)
+	(global_label "PWM_2"
+		(shape output)
+		(at 170.18 99.06 180)
+		(fields_autoplaced yes)
+		(effects
+			(font
+				(size 1.27 1.27)
+			)
+			(justify right)
+		)
+		(property "Intersheetrefs" "${INTERSHEET_REFS}"
+			(at 160.8449 99.06 0)
+			(effects
+				(font
+					(size 1.27 1.27)
+				)
+				(justify right)
 				(hide yes)
 			)
@@
 		)
 	)
-	(global_label "PWM_2"
-		(shape output)
-		(at 222.25 111.76 0)
-		(fields_autoplaced yes)
-		(effects
-			(font
-				(size 1.27 1.27)
-			)
-			(justify left)
-		)
-		(property "Intersheetrefs" "${INTERSHEET_REFS}"
-			(at 231.5851 111.76 0)
-			(effects
-				(font
-					(size 1.27 1.27)
-				)
-				(justify left)
+	(global_label "PWM_1"
+		(shape output)
+		(at 170.18 96.52 180)
+		(fields_autoplaced yes)
+		(effects
+			(font
+				(size 1.27 1.27)
+			)
+			(justify right)
+		)
+		(property "Intersheetrefs" "${INTERSHEET_REFS}"
+			(at 160.8449 96.52 0)
+			(effects
+				(font
+					(size 1.27 1.27)
+				)
+				(justify right)
 				(hide yes)
 			)
@@
 		)
 	)
-	(global_label "PWM_4"
-		(shape output)
-		(at 222.25 119.38 0)
-		(fields_autoplaced yes)
-		(effects
-			(font
-				(size 1.27 1.27)
-			)
-			(justify left)
-		)
-		(property "Intersheetrefs" "${INTERSHEET_REFS}"
-			(at 231.5851 119.38 0)
-			(effects
-				(font
-					(size 1.27 1.27)
-				)
-				(justify left)
-				(hide yes)
-			)
-		)
-	)
 	(global_label "SENSOR_INT"
 		(shape input)
@@
 			(effects
 				(font
-					(size 1.27 1.27)
-				)
-				(justify left)
-				(hide yes)
-			)
-		)
-	)
-	(global_label "PWM_1"
-		(shape output)
-		(at 222.25 114.3 0)
-		(fields_autoplaced yes)
-		(effects
-			(font
-				(size 1.27 1.27)
-			)
-			(justify left)
-		)
-		(property "Intersheetrefs" "${INTERSHEET_REFS}"
-			(at 231.5851 114.3 0)
-			(effects
-				(font
